File: hardware/riffle-CTL-0.2-throughhole.sch (EAGLE design)
At the start: 14 parts, among them J2 AYZ0202

Commit message: update
Parts:
- removed 555: NE555D, SparkFun-AnalogIC:NE555D
- removed EC: 1X2-3.5MM, adafruit:1X2-3.5MM
- removed J2: AYZ0202, SparkFunNew:AYZ0202
- removed R2: 10k, rcl:R-EU_R0805
- added EC1: 1X2-3.5MM, adafruit:1X2-3.5MM
- added IC1: LM555N, linear:LM555N
- added R1: 10k, resistor:R-EU_0204/7
- added SV1: (no value), con-lstb:MA03-1
- C1, C7: value 1uF -> 10µ; device resistor:C-EUC0805 -> resistor:CPOL-EUE1.8-4
- C2: value .1uF -> .1; device resistor:C-EUC0805 -> resistor:CPOL-EUE1.8-4
- C3: value .01u -> 0.01µ; device resistor:C-EUC0805 -> resistor:C-EU025-024X044
- C4: value 100n -> 0.1µ; device resistor:C-EUC0805 -> resistor:C-EU025-024X044
- C5: value 100n -> .1µ; device resistor:C-EUC0805 -> resistor:CPOL-EUE1.8-4
- C6: value .1uF -> 1u; device resistor:C-EUC0805 -> resistor:CPOL-EUE1.8-4
Connections:
- removed net N$2: 555.CON, C3.2
- removed net N$6: C2.1, J2.1, J2.4
- removed net N1: 555.TRE, 555.TRI, EC.1, J2.2, J2.5
- removed net VDD2: C1.1, J2.3, J2.6
- new net N$1: C1.+, SV1.3
- new net N$3: EC1.1, IC1.THR, IC1.TR, SV1.2
- new net N$4: C2.+, SV1.1
- new net N$7: C3.2, IC1.CV
- net EC: now also EC1.2, IC1.Q; no longer 555.OUT, EC.2
- net GND: now also C1.-, C2.-, C4.2, C5.-, C6.-, C7.-, IC1.GND; no longer 555.GND, C1.2, C2.2, C4.1, C5.1, C6.1, C7.1
- net THRM: now also R1.1; no longer R2.1
- net VCC: now also C4.1, C5.+, C6.+, C7.+, IC1.R, IC1.V+, R1.2; no longer 555./RES, 555.VCC+, C4.2, C5.2, C6.2, C7.2, R2.2
Other:
- moved on the sheet: C3, C4
