File: hardware/riffle-CTL-0.3-cap.brd (EAGLE design)
At the start: 18.4 x 18.4 mm, 12 parts

Commit message: update
Parts:
- moved G 1.40 mm to (17.5, 11.7)
- moved E1 1.40 mm to (18.8, 14.2)
- moved E1A 1.40 mm to (21.5, 14.2)
- moved E2 1.40 mm to (18.8, 16.9)
- moved E2A 1.40 mm to (21.5, 16.9)
Routing:
- net N$2: track 7.85 -> 9.25 mm
Other:
- board outline removed
- board text added: "CT-0.3"
- board text added: "publiclab.org/wiki/coqui"
Changed lines of the file:
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@@
 <plain>
 <wire x1="7.62" y1="14.605" x2="7.62" y2="14.478" width="0" layer="20"/>
-<wire x1="7.62" y1="14.478" x2="7.62" y2="14.605" width="0" layer="20" curve="359.209763"/>
+<wire x1="7.62" y1="14.478" x2="7.62" y2="14.605" width="0" layer="22" curve="359.209763"/>
+<text x="16.637" y="6.35" size="1.27" layer="21" rot="R20">CT-0.3</text>
+<text x="25.654" y="12.827" size="0.8128" layer="22" font="vector" rot="MR340">publiclab.org/wiki/coqui</text>
 </plain>
 <attributes>
@@
 </autorouter>
 <elements>
-<element name="1W" library="pinhead" package="1X01" value="" x="16.129" y="14.224"/>
-<element name="E1" library="pinhead" package="1X01" value="" x="18.796" y="12.827" rot="R180"/>
-<element name="E2" library="pinhead" package="1X01" value="" x="18.796" y="15.494"/>
-<element name="PA" library="pinhead" package="1X01" value="" x="13.462" y="16.891" rot="R90"/>
-<element name="GA" library="pinhead" package="1X01" value="" x="13.462" y="11.557" rot="R180"/>
-<element name="E1A" library="pinhead" package="1X01" value="" x="21.463" y="12.827" rot="R270"/>
-<element name="E2A" library="pinhead" package="1X01" value="" x="21.463" y="15.494"/>
-<element name="P" library="pinhead" package="1X01" value="" x="16.129" y="16.891" rot="R90"/>
-<element name="G" library="pinhead" package="1X01" value="" x="16.129" y="11.557" rot="R180"/>
-<element name="1WA" library="pinhead" package="1X01" value="" x="13.462" y="14.224" rot="R90"/>
-<element name="RA" library="pinhead" package="1X01" value="" x="10.795" y="15.621"/>
-<element name="RB" library="pinhead" package="1X01" value="" x="14.859" y="19.431"/>
+<element name="1W" library="pinhead" package="1X01" value="" x="16.129" y="14.224" smashed="yes">
+<attribute name="NAME" x="15.9258" y="10.9728" size="1.016" layer="25" ratio="10" rot="R90"/>
+<attribute name="VALUE" x="14.859" y="11.049" size="1.27" layer="27"/>
+</element>
+<element name="E1" library="pinhead" package="1X01" value="" x="18.796" y="14.224" smashed="yes" rot="R180">
+<attribute name="NAME" x="19.3802" y="12.2682" size="1.016" layer="25" ratio="10" rot="R315"/>
+<attribute name="VALUE" x="20.066" y="17.399" size="1.27" layer="27" rot="R180"/>
+</element>
+<element name="E2" library="pinhead" package="1X01" value="" x="18.796" y="16.891" smashed="yes">
+<attribute name="NAME" x="18.5928" y="18.4658" size="1.016" layer="25" ratio="10"/>
+<attribute name="VALUE" x="17.526" y="13.716" size="1.27" layer="27"/>
+</element>
+<element name="PA" library="pinhead" package="1X01" value="" x="13.462" y="16.891" smashed="yes" rot="R90">
+<attribute name="NAME" x="12.3952" y="18.9992" size="1.016" layer="25" ratio="10" rot="R180"/>
+<attribute name="VALUE" x="16.637" y="15.621" size="1.27" layer="27" rot="R90"/>
+</element>
+<element name="GA" library="pinhead" package="1X01" value="" x="13.462" y="11.557" smashed="yes" rot="R180">
+<attribute name="NAME" x="12.5222" y="10.1092" size="1.016" layer="25" ratio="10" rot="R180"/>
+<attribute name="VALUE" x="14.732" y="14.732" size="1.27" layer="27" rot="R180"/>
+</element>
+<element name="E1A" library="pinhead" package="1X01" value="" x="21.463" y="14.224" smashed="yes" rot="R270">
+<attribute name="NAME" x="24.2062" y="12.7508" size="1.016" layer="25" ratio="10" rot="R90"/>
+<attribute name="VALUE" x="18.288" y="15.494" size="1.27" layer="27" rot="R270"/>
+</element>
+<element name="E2A" library="pinhead" package="1X01" value="" x="21.463" y="16.891" smashed="yes">
+<attribute name="NAME" x="21.1328" y="18.4658" size="1.016" layer="25" ratio="10"/>
+<attribute name="VALUE" x="20.193" y="13.716" size="1.27" layer="27"/>
+</element>
+<element name="P" library="pinhead" package="1X01" value="" x="16.129" y="16.891" smashed="yes" rot="R90">
+<attribute name="NAME" x="17.6022" y="19.3802" size="1.016" layer="25" ratio="10" rot="R180"/>
+<attribute name="VALUE" x="19.304" y="15.621" size="1.27" layer="27" rot="R90"/>
+</element>
+<element name="G" library="pinhead" package="1X01" value="" x="17.526" y="11.684" smashed="yes" rot="R180">
+<attribute name="NAME" x="17.9832" y="9.9822" size="1.016" layer="25" ratio="10" rot="R180"/>
+<attribute name="VALUE" x="18.796" y="14.859" size="1.27" layer="27" rot="R180"/>
+</element>
+<element name="1WA" library="pinhead" package="1X01" value="" x="13.462" y="14.224" smashed="yes" rot="R90">
+<attribute name="NAME" x="12.0142" y="13.7922" size="1.016" layer="25" ratio="10" rot="R180"/>
+<attribute name="VALUE" x="16.637" y="12.954" size="1.27" layer="27" rot="R90"/>
+</element>
+<element name="RA" library="pinhead" package="1X01" value="" x="10.795" y="15.621" smashed="yes">
+<attribute name="NAME" x="9.0932" y="14.7828" size="1.016" layer="25" ratio="10" rot="R90"/>
+<attribute name="VALUE" x="9.525" y="12.446" size="1.27" layer="27"/>
+</element>
+<element name="RB" library="pinhead" package="1X01" value="" x="14.859" y="19.431" smashed="yes">
+<attribute name="NAME" x="14.1478" y="21.2598" size="1.016" layer="25" ratio="10"/>
+<attribute name="VALUE" x="13.589" y="16.256" size="1.27" layer="27"/>
+</element>
 </elements>
 <signals>
@@
 <wire x1="16.0528" y1="11.5824" x2="13.6144" y2="11.5824" width="0.2032" layer="1"/>
 <wire x1="13.6144" y1="11.5824" x2="13.462" y2="11.557" width="0.2032" layer="1"/>
-<wire x1="16.0528" y1="11.5824" x2="16.129" y2="11.557" width="0.2032" layer="1"/>
+<wire x1="16.0528" y1="11.5824" x2="17.526" y2="11.684" width="0.2032" layer="1"/>
 <wire x1="10.9728" y1="14.0208" x2="10.9728" y2="15.4432" width="0.2032" layer="1"/>
 <wire x1="13.4112" y1="11.5824" x2="10.9728" y2="14.0208" width="0.2032" layer="1"/>
@@
 <contactref element="E1" pad="1"/>
 <contactref element="E1A" pad="1"/>
-<wire x1="21.336" y1="12.8016" x2="18.8976" y2="12.8016" width="0.2032" layer="1"/>
-<wire x1="18.8976" y1="12.8016" x2="18.796" y2="12.827" width="0.2032" layer="1"/>
-<wire x1="21.336" y1="12.8016" x2="21.463" y2="12.827" width="0.2032" layer="1"/>
+<wire x1="21.336" y1="14.1986" x2="18.8976" y2="14.1986" width="0.2032" layer="1"/>
+<wire x1="18.8976" y1="14.1986" x2="18.796" y2="14.224" width="0.2032" layer="1"/>
+<wire x1="21.336" y1="14.1986" x2="21.463" y2="14.224" width="0.2032" layer="1"/>
 </signal>
 <signal name="N$5">
 <contactref element="E2" pad="1"/>
 <contactref element="E2A" pad="1"/>
-<wire x1="21.336" y1="15.4432" x2="18.8976" y2="15.4432" width="0.2032" layer="1"/>
-<wire x1="18.8976" y1="15.4432" x2="18.796" y2="15.494" width="0.2032" layer="1"/>
-<wire x1="21.336" y1="15.4432" x2="21.463" y2="15.494" width="0.2032" layer="1"/>
+<wire x1="21.336" y1="16.8402" x2="18.8976" y2="16.8402" width="0.2032" layer="1"/>
+<wire x1="18.8976" y1="16.8402" x2="18.796" y2="16.891" width="0.2032" layer="1"/>
+<wire x1="21.336" y1="16.8402" x2="21.463" y2="16.891" width="0.2032" layer="1"/>
 </signal>
 </signals>

Commit message: update
Parts:
- moved 1W 9.55 mm to (8.38, 8.64)
- moved E1A 9.55 mm to (13.7, 8.64)
- moved 1WA 9.55 mm to (5.71, 8.64)
- moved E1 9.55 mm to (11.0, 8.64)
- moved G 9.55 mm to (9.78, 6.10)
- moved GA 9.55 mm to (5.71, 5.97)
- moved RA 9.55 mm to (3.05, 10.0)
- moved RB 9.55 mm to (7.11, 13.8)
- moved E2 9.55 mm to (11.0, 11.3)
- moved E2A 9.55 mm to (13.7, 11.3)
- moved P 9.55 mm to (8.38, 11.3)
- moved PA 9.55 mm to (5.71, 11.3)
Other:
- board outline added: 18.4 x 18.4 mm
